Commit message: train cyberdog2

File: resources/cyberdog2/urdf/cyberdog2.urdf (robot description, URDF)
Before this commit: robot cyberdog2, 40 links, 39 joints
Links:
- removed link AI_camera_link
- removed link D435_camera_link
- removed link FL_abad
- removed link FL_abad_rotor
- removed link FL_hip_rotor
- removed link FL_hip_shoulder
- removed link FL_knee
- removed link FL_knee_rotor
- removed link FR_abad
- removed link FR_abad_rotor
- removed link FR_hip_rotor
- removed link FR_hip_shoulder
- removed link FR_knee
- removed link FR_knee_rotor
- removed link RGB_camera_link
- removed link RL_abad
- removed link RL_abad_rotor
- removed link RL_hip_rotor
- removed link RL_hip_shoulder
- removed link RL_knee
- removed link RL_knee_rotor
- removed link RR_abad
- removed link RR_abad_rotor
- removed link RR_hip_rotor
- removed link RR_hip_shoulder
- removed link RR_knee
- removed link RR_knee_rotor
- removed link body
- removed link head
- removed link imu_link
- removed link lidar_link
- added link FL_battery
- added link FL_calf, mass 0.116; collision box size=0.016 0.016 0.18341; visual mesh filename=../meshes/knee.stl scale=1 1 1
- added link FL_thigh, mass 0.482; visual mesh filename=../meshes/hip.stl scale=1 1 1
- added link FR_battery
- added link FR_calf, mass 0.116; collision box size=0.016 0.016 0.18341; visual mesh filename=../meshes/knee.stl scale=1 1 1
- added link FR_thigh, mass 0.482; visual mesh filename=../meshes/hip_mirror.stl scale=1 1 1
- added link RL_battery
- added link RL_calf, mass 0.116; collision box size=0.016 0.016 0.18341; visual mesh filename=../meshes/knee.stl scale=1 1 1
- added link RL_thigh, mass 0.482; visual mesh filename=../meshes/hip.stl scale=1 1 1
- added link RR_battery
- added link RR_calf, mass 0.116; collision box size=0.016 0.016 0.18341; visual mesh filename=../meshes/knee.stl scale=1 1 1
- added link RR_thigh, mass 0.482; visual mesh filename=../meshes/hip_mirror.stl scale=1 1 1
- link FL_foot: mass None -> 0.004; geometry collision sphere radius=0.02; visual sphere radius=0.01
- link FL_hip: mass 0.482 -> 0.354; geometry collision cylinder length=0.035 radius=0.039; visual mesh filename=../meshes/abad.stl scale=1 1 1
- link FR_foot: mass None -> 0.004; geometry collision sphere radius=0.02; visual sphere radius=0.01
- link FR_hip: mass 0.482 -> 0.354; geometry collision cylinder length=0.035 radius=0.039; visual mesh filename=../meshes/abad.stl scale=1 1 1
- link RL_foot: mass None -> 0.004; geometry collision sphere radius=0.02; visual sphere radius=0.01
- link RL_hip: mass 0.482 -> 0.354; geometry collision cylinder length=0.035 radius=0.039; visual mesh filename=../meshes/abad.stl scale=1 1 1
- link RR_foot: mass None -> 0.004; geometry collision sphere radius=0.02; visual sphere radius=0.01
- link RR_hip: mass 0.482 -> 0.354; geometry collision cylinder length=0.035 radius=0.039; visual mesh filename=../meshes/abad.stl scale=1 1 1
- link base: mass None -> 4.03; geometry collision box size=0.4 0.25 0.109; visual mesh filename=../meshes/body.stl scale=1 1 1
Joints:
- removed joint AI_camera_joint
- removed joint D435_camera_joint
- removed joint FL_abad_fixed
- removed joint FL_abad_joint
- removed joint FL_abad_rotor_fix
- removed joint FL_foot_fixed
- removed joint FL_hip_rotor_fix
- removed joint FL_knee_joint
- removed joint FL_knee_rotor_fix
- removed joint FR_abad_fixed
- removed joint FR_abad_joint
- removed joint FR_abad_rotor_fix
- removed joint FR_foot_fixed
- removed joint FR_hip_rotor_fix
- removed joint FR_knee_joint
- removed joint FR_knee_rotor_fix
- removed joint RGB_camera_joint
- removed joint RL_abad_fixed
- removed joint RL_abad_joint
- removed joint RL_abad_rotor_fix
- removed joint RL_foot_fixed
- removed joint RL_hip_rotor_fix
- removed joint RL_knee_joint
- removed joint RL_knee_rotor_fix
- removed joint RR_abad_fixed
- removed joint RR_abad_joint
- removed joint RR_abad_rotor_fix
- removed joint RR_foot_fixed
- removed joint RR_hip_rotor_fix
- removed joint RR_knee_joint
- removed joint RR_knee_rotor_fix
- removed joint floating_base
- removed joint head_joint
- removed joint imu_joint
- removed joint scan_joint
- added joint FL_calf_joint: type revolute, parent FL_thigh, child FL_calf, origin xyz=0 0 -0.12 rpy=0 0 0, axis 0 1 0, limit lower=-2.5307274153917776 upper=-0.5235987755982988 effort=12.0001 velocity=30.9971
- added joint FL_foot_joint: type fixed, parent FL_calf, child FL_foot, origin xyz=0 0 -0.18341 rpy=0 0 0, axis 0 1 0
- added joint FL_thigh_joint: type revolute, parent FL_hip, child FL_thigh, origin xyz=0 0.094 0 rpy=0 0 0, axis 0 1 0, limit lower=-1.3264502315156903 upper=2.792526803190927 effort=12.0001 velocity=30.9971
- added joint FR_calf_joint: type revolute, parent FR_thigh, child FR_calf, origin xyz=0 0 -0.12 rpy=0 0 0, axis 0 1 0, limit lower=-2.5307274153917776 upper=-0.5235987755982988 effort=12.0001 velocity=30.9971
- added joint FR_foot_joint: type fixed, parent FR_calf, child FR_foot, origin xyz=0 0 -0.18341 rpy=0 0 0, axis 0 1 0
- added joint FR_thigh_joint: type revolute, parent FR_hip, child FR_thigh, origin xyz=0 -0.094 0 rpy=0 0 0, axis 0 1 0, limit lower=-1.3264502315156903 upper=2.792526803190927 effort=12.0001 velocity=30.9971
- added joint RL_calf_joint: type revolute, parent RL_thigh, child RL_calf, origin xyz=0 0 -0.12 rpy=0 0 0, axis 0 1 0, limit lower=-2.5307274153917776 upper=-0.5235987755982988 effort=12.0001 velocity=30.9971
- added joint RL_foot_joint: type fixed, parent RL_calf, child RL_foot, origin xyz=0 0 -0.18341 rpy=0 1 0
- added joint RL_thigh_joint: type revolute, parent RL_hip, child RL_thigh, origin xyz=0 0.094 0 rpy=0 0 0, axis 0 1 0, limit lower=-0.9773843811168246 upper=3.141592653589793 effort=12.0001 velocity=30.9971
- added joint RR_calf_joint: type revolute, parent RR_thigh, child RR_calf, origin xyz=0 0 -0.12 rpy=0 0 0, axis 0 1 0, limit lower=-2.5307274153917776 upper=-0.5235987755982988 effort=12.0001 velocity=30.9971
- added joint RR_foot_joint: type fixed, parent RR_calf, child RR_foot, origin xyz=0 0 -0.18341 rpy=0 1 0
- added joint RR_thigh_joint: type revolute, parent RR_hip, child RR_thigh, origin xyz=0 -0.094 0 rpy=0 0 0, axis 0 1 0, limit lower=-0.9773843811168246 upper=3.141592653589793 effort=12.0001 velocity=30.9971
- added joint battery_joint_fl: type fixed, parent base, child FL_battery, origin xyz=0.09775 0.07 0 rpy=0 0 0, axis 0 0 0
- added joint battery_joint_fr: type fixed, parent base, child FR_battery, origin xyz=0.09775 -0.07 0 rpy=0 0 0, axis 0 0 0
- added joint battery_joint_rl: type fixed, parent base, child RL_battery, origin xyz=-0.09775 0.07 0 rpy=0 0 0, axis 0 0 0
- added joint battery_joint_rr: type fixed, parent base, child RR_battery, origin xyz=-0.09775 -0.07 0 rpy=0 0 0, axis 0 0 0
- joint FL_hip_joint: axis 0 1 0 -> 1 0 0; limit lower=-1.3264502315156903 upper=2.792526803190927 effort=12.0001 velocity=30.9971 -> lower=-0.6806784082777885 upper=0.6806784082777885 effort=12.0001 velocity=30.9971; origin xyz=0 0.094 0 rpy=0 0 0 -> xyz=0.164 0.042 0 rpy=0 0 0; parent FL_abad -> base
- joint FR_hip_joint: axis 0 1 0 -> 1 0 0; limit lower=-1.3264502315156903 upper=2.792526803190927 effort=12.0001 velocity=30.9971 -> lower=-0.6806784082777885 upper=0.6806784082777885 effort=12.0001 velocity=30.9971; origin xyz=0 -0.094 0 rpy=0 0 0 -> xyz=0.164 -0.042 0 rpy=0 0 0; parent FR_abad -> base
- joint RL_hip_joint: axis 0 1 0 -> 1 0 0; limit lower=-0.9773843811168246 upper=3.141592653589793 effort=12.0001 velocity=30.9971 -> lower=-0.6806784082777885 upper=0.6806784082777885 effort=12.0001 velocity=30.9971; origin xyz=0 0.094 0 rpy=0 0 0 -> xyz=-0.164 0.042 0 rpy=0 0 0; parent RL_abad -> base
- joint RR_hip_joint: axis 0 1 0 -> 1 0 0; limit lower=-0.9773843811168246 upper=3.141592653589793 effort=12.0001 velocity=30.9971 -> lower=-0.6806784082777885 upper=0.6806784082777885 effort=12.0001 velocity=30.9971; origin xyz=0 -0.094 0 rpy=0 0 0 -> xyz=-0.164 -0.042 0 rpy=0 0 0; parent RR_abad -> base

Commit message: train 0.2 height

File: resources/cyberdog2/urdf/cyberdog2.urdf (robot description, URDF)
Before this commit: robot titatit_robot_2, 21 links, 20 joints
Links:
- link FL_calf: geometry collision box size=0.016 0.016 0.18341; visual box size=0.016 0.016 0.18341
- link FL_foot: geometry collision sphere radius=0.02; visual sphere radius=0.02
- link FR_calf: geometry collision box size=0.016 0.016 0.18341; visual box size=0.016 0.016 0.18341
- link FR_foot: geometry collision sphere radius=0.02; visual sphere radius=0.02
- link RL_calf: geometry collision box size=0.016 0.016 0.18341; visual box size=0.016 0.016 0.18341
- link RL_foot: geometry collision sphere radius=0.02; visual sphere radius=0.02
- link RR_calf: geometry collision box size=0.016 0.016 0.18341; visual box size=0.016 0.016 0.18341
- link RR_foot: geometry collision sphere radius=0.02; visual sphere radius=0.02
